File: circuit_schematics/LPC1347_shield/shield.brd (EAGLE design)
At the start: 17 parts, among them IC1 7805TV, IC2 LD1117V33

Commit message: Fixed isolation on ground pour.
Routing:
- net GND: track 183.5 -> 181.0 mm
Changed lines of the file:
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@@
 <wire x1="7.6962" y1="18.9738" x2="8.89" y2="17.78" width="0.254" layer="16"/>
 <wire x1="24.13" y1="8.89" x2="25.4" y2="10.16" width="0.254" layer="16"/>
-<wire x1="25.4" y1="10.16" x2="25.4" y2="15.24" width="0.254" layer="16"/>
-<wire x1="25.4" y1="15.24" x2="26.67" y2="16.51" width="0.254" layer="16"/>
+<wire x1="25.4" y1="10.16" x2="25.4" y2="16.51" width="0.254" layer="16"/>
 <wire x1="65.405" y1="20.955" x2="61.595" y2="20.955" width="0.254" layer="16"/>
 <wire x1="61.595" y1="20.955" x2="59.69" y2="22.86" width="0.254" layer="16"/>
@@
 <wire x1="69.215" y1="20.955" x2="72.39" y2="17.78" width="0.254" layer="16"/>
 <wire x1="72.39" y1="17.78" x2="87.63" y2="17.78" width="0.254" layer="16"/>
-<wire x1="36.83" y1="16.51" x2="26.67" y2="16.51" width="0.254" layer="16"/>
+<wire x1="36.83" y1="16.51" x2="35.56" y2="16.51" width="0.254" layer="16"/>
+<wire x1="35.56" y1="16.51" x2="26.67" y2="16.51" width="0.254" layer="16"/>
 <wire x1="59.69" y1="22.86" x2="59.69" y2="21.59" width="0.254" layer="16"/>
 <wire x1="59.69" y1="21.59" x2="58.42" y2="20.32" width="0.254" layer="16"/>
@@
 <wire x1="45.72" y1="24.13" x2="45.72" y2="24.765" width="0.254" layer="16"/>
 <wire x1="45.72" y1="24.765" x2="44.45" y2="26.035" width="0.254" layer="16"/>
-<wire x1="44.45" y1="26.035" x2="36.195" y2="26.035" width="0.254" layer="16"/>
-<wire x1="36.195" y1="26.035" x2="26.67" y2="16.51" width="0.254" layer="16"/>
+<wire x1="44.45" y1="26.035" x2="35.56" y2="26.035" width="0.254" layer="16"/>
 <wire x1="45.72" y1="10.16" x2="45.72" y2="13.97" width="0.254" layer="16"/>
 <wire x1="45.72" y1="13.97" x2="45.72" y2="20.32" width="0.254" layer="16"/>
@@
 <wire x1="90.17" y1="10.16" x2="87.63" y2="12.7" width="0.254" layer="16"/>
 <wire x1="87.63" y1="17.78" x2="87.63" y2="12.7" width="0.254" layer="16"/>
-<polygon width="0.4064" layer="16">
+<polygon width="0.4064" layer="16" isolate="0.3048">
 <vertex x="-1.27" y="35.56"/>
 <vertex x="-1.27" y="0"/>
@@
 <vertex x="95.25" y="35.56"/>
 </polygon>
+<wire x1="25.4" y1="16.51" x2="26.67" y2="16.51" width="0.254" layer="16"/>
+<wire x1="35.56" y1="26.035" x2="35.56" y2="16.51" width="0.254" layer="16"/>
 </signal>
 <signal name="+3V3">
@@
 <contactref element="PROGRAM_SW" pad="1"/>
 <wire x1="8.255" y1="4.445" x2="8.89" y2="3.81" width="0.254" layer="16"/>
-<wire x1="8.89" y1="3.81" x2="40.64" y2="3.81" width="0.254" layer="16"/>
 <wire x1="40.64" y1="3.81" x2="42.545" y2="5.715" width="0.254" layer="16"/>
 <wire x1="7.6962" y1="10.4394" x2="7.6962" y2="6.9088" width="0.254" layer="16"/>
 <wire x1="7.6962" y1="6.9088" x2="8.255" y2="6.35" width="0.254" layer="16"/>
 <wire x1="8.255" y1="6.35" x2="8.255" y2="4.445" width="0.254" layer="16"/>
+<wire x1="40.64" y1="3.81" x2="8.89" y2="3.81" width="0.254" layer="16"/>
 </signal>
 <signal name="PIO0_5">

Commit message: Fixed Wiring Error.
Wire from ESP8266 RX must go to P0_19 not P1_19.
Connections:
- net PIO0_19: now also LPC1.9; no longer LPC1.12
Routing:
- net PIO0_19: track 15.5 -> 13.8 mm
Changed lines of the file:
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@@
 <wire x1="87.63" y1="17.78" x2="87.63" y2="12.7" width="0.254" layer="16"/>
 <polygon width="0.4064" layer="16" isolate="0.3048">
-<vertex x="-1.27" y="35.56"/>
-<vertex x="-1.27" y="0"/>
-<vertex x="95.25" y="0"/>
-<vertex x="95.25" y="35.56"/>
+<vertex x="-3.81" y="35.56"/>
+<vertex x="-3.81" y="0"/>
+<vertex x="143.51" y="0"/>
+<vertex x="143.51" y="35.56"/>
 </polygon>
 <wire x1="25.4" y1="16.51" x2="26.67" y2="16.51" width="0.254" layer="16"/>
@@
 </signal>
 <signal name="PIO0_19">
-<contactref element="LPC1" pad="12"/>
 <contactref element="ESP8266" pad="1"/>
 <wire x1="52.07" y1="22.86" x2="49.53" y2="25.4" width="0.254" layer="16"/>
 <wire x1="49.53" y1="25.4" x2="49.53" y2="27.305" width="0.254" layer="16"/>
 <wire x1="49.53" y1="27.305" x2="41.275" y2="27.305" width="0.254" layer="16"/>
-<wire x1="41.275" y1="27.305" x2="40.005" y2="28.575" width="0.254" layer="16"/>
+<contactref element="LPC1" pad="9"/>
+<wire x1="49.53" y1="27.305" x2="47.625" y2="28.575" width="0" layer="19" extent="16-16"/>
 </signal>
 <signal name="PIO0_13">
